File: GEMS_Amethyst/GEMS_Amethyst.kicad_sch (KiCad schematic)
At the start: 37 parts, among them J1 RGB, J2 LX, J3 I2C, J4 UART, J5 USB_C_USB2.0, Q1 TEPT5700, SW1 BTN, SW2 RST, U1 ESP32-C3, U2 R1170H331B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

Commit message: updated Library
Parts:
- C1, C2, C3, C4, C5, C6, C7, C8: footprint GEMS_library:C_1206_(3216) -> GEMS_Library:C_1206_(3216); symbol GEMS_library:Capacitor -> GEMS_Library:Capacitor
- D1: footprint GEMS_library:LED_D5.0mm-4_RGB -> GEMS_Library:LED_D5.0mm-4_RGB; symbol GEMS_library:LED_BkRG -> GEMS_Library:LED_BkRG
- J1, J2, J3, J4: footprint GEMS_library:PinHeader_1x04_P2.54mm_Vertical -> GEMS_Library:PinHeader_1x04_P2.54mm_Vertical; symbol GEMS_library:Conn_01x04 -> GEMS_Library:Conn_01x04
- J5: footprint GEMS_library:USB-C_MOLEX-216990-0001 -> GEMS_Library:USB-C_MOLEX-216990-0001; symbol GEMS_library:USB_C_USB2.0 -> GEMS_Library:USB_C_USB2.0
- Q1: footprint GEMS_library:PT_D5.0mm -> GEMS_Library:PT_D5.0mm; symbol GEMS_library:TEPT5700 -> GEMS_Library:TEPT5700
- R1, R10, R11, R12, R13, R14, R15, R16, R17, R2, R3, R4, R5, R6, R7, R8, R9: footprint GEMS_library:R_1206_(3216) -> GEMS_Library:R_1206_(3216); symbol GEMS_library:Resistor -> GEMS_Library:Resistor
- SW1, SW2: footprint GEMS_library:SW_PUSH_6mm_SMD -> GEMS_Library:SW_PUSH_6mm_SMD; symbol GEMS_library:SW_Push_NO -> GEMS_Library:SW_Push_NO
- U1: footprint GEMS_library:ESP32-C3-WROOM-02 -> GEMS_Library:ESP32-C3-WROOM-02; symbol GEMS_library:ESP32-C3 -> GEMS_Library:ESP32-C3
- U2: footprint GEMS_library:SOT-89-5 -> GEMS_Library:SOT-89-5; symbol GEMS_library:R1170H331B -> GEMS_Library:R1170H331B
- U3: footprint GEMS_library:SOT-23-6 -> GEMS_Library:SOT-23-6; symbol GEMS_library:USBLC6-2SC6 -> GEMS_Library:USBLC6-2SC6
