File: GEMS_Diamond/GEMS_Diamond.kicad_sch (KiCad schematic)
At the start: 46 parts, among them J1 USB_C_USB2.0, J2 ConnScrew_01x16, Q1 DMG2305UX-13, SW1 BTN, SW2 RST, U1 R1170H331B, U2 ESP32-S3-WROOM, U3 USBLC6-2SC6, U4 DRV8411, U5 ACS71240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

Commit message: updated Library
Parts:
- C1, C10, C11, C12, C2, C3, C4, C5, C6, C7, C8, C9: footprint GEMS_library:C_1206_(3216) -> GEMS_Library:C_1206_(3216); symbol GEMS_library:Capacitor -> GEMS_Library:Capacitor
- CAN1, CAN2: footprint GEMS_library:IDC8_Micro-MaTch -> GEMS_Library:IDC8_Micro-MaTch; symbol GEMS_library:CAN_connector -> GEMS_Library:CAN_connector
- D1: footprint GEMS_library:DO-214_(SMA) -> GEMS_Library:DO-214_(SMA); symbol GEMS_library:XBS306 -> GEMS_Library:XBS306
- D2, D3, D4, D5: footprint GEMS_library:LED_D3.0mm -> GEMS_Library:LED_D3.0mm; symbol GEMS_library:LED -> GEMS_Library:LED
- J1: footprint GEMS_library:USB-C_MOLEX-216990-0001 -> GEMS_Library:USB-C_MOLEX-216990-0001; symbol GEMS_library:USB_C_USB2.0 -> GEMS_Library:USB_C_USB2.0
- J2: footprint GEMS_library:TerminalScrew_1x16_P3.5mm -> GEMS_Library:TerminalScrew_1x16_P3.5mm; symbol GEMS_library:ConnScrew_01x16 -> GEMS_Library:ConnScrew_01x16
- Q1: footprint GEMS_library:SOT-23 -> GEMS_Library:SOT-23; symbol GEMS_library:DMG2305UX-13 -> GEMS_Library:DMG2305UX-13
- R1, R10, R11, R12, R13, R14, R15, R16, R2, R3, R4, R5, R6, R7, R8, R9: footprint GEMS_library:R_1206_(3216) -> GEMS_Library:R_1206_(3216); symbol GEMS_library:Resistor -> GEMS_Library:Resistor
- SW1, SW2: footprint GEMS_library:SW_PUSH_6mm_SMD -> GEMS_Library:SW_PUSH_6mm_SMD; symbol GEMS_library:SW_Push_NO -> GEMS_Library:SW_Push_NO
- U1: footprint GEMS_library:SOT-89-5 -> GEMS_Library:SOT-89-5; symbol GEMS_library:R1170H331B -> GEMS_Library:R1170H331B
- U2: footprint GEMS_library:ESP32-S3-WROOM -> GEMS_Library:ESP32-S3-WROOM; symbol GEMS_library:ESP32-S3-WROOM -> GEMS_Library:ESP32-S3-WROOM
- U3: footprint GEMS_library:SOT-23-6 -> GEMS_Library:SOT-23-6; symbol GEMS_library:USBLC6-2SC6 -> GEMS_Library:USBLC6-2SC6
- U4: footprint GEMS_library:HTSSOP-16_4.4x5mm_P0.65mm -> GEMS_Library:HTSSOP-16_4.4x5mm_P0.65mm; symbol GEMS_library:DRV8411 -> GEMS_Library:DRV8411
- U5: footprint GEMS_library:SOIC-8 -> GEMS_Library:SOIC-8; symbol GEMS_library:ACS71240 -> GEMS_Library:ACS71240
- U6: footprint GEMS_library:SOIC-8 -> GEMS_Library:SOIC-8; symbol GEMS_library:TCAN332DR -> GEMS_Library:TCAN332DR
