File: GEMS_Emerald/GEMS_Emerald.kicad_sch (KiCad schematic)
At the start: 68 parts, among them J1 USB_C_USB2.0, J2 18650_battery_holder, Q1 DMG2305UX-13, Q2 DMP3036SSD-13, Q3 BC846, Q4 BC846, Q5 DMN2310U, SW1 BTN, SW2 RST, SW3 EN, SW4 SW_SPDT, U1 R1170H331B, U2 ESP32-C3, U3 USBLC6-2SC6, U4 MCP6002, U5 MCP73831T, U6 TCAN332DR

Commit message: updated Library
Parts:
- C1, C10, C11, C12, C13, C2, C3, C4, C5, C6, C7, C8, C9: footprint GEMS_library:C_1206_(3216) -> GEMS_Library:C_1206_(3216); symbol GEMS_library:Capacitor -> GEMS_Library:Capacitor
- CAN1, CAN2: footprint GEMS_library:IDC8_Micro-MaTch -> GEMS_Library:IDC8_Micro-MaTch; symbol GEMS_library:CAN_connector -> GEMS_Library:CAN_connector
- D1: footprint GEMS_library:DO-214_(SMA) -> GEMS_Library:DO-214_(SMA); symbol GEMS_library:XBS306 -> GEMS_Library:XBS306
- D2, D3, D4, D5: footprint GEMS_library:LED_D3.0mm -> GEMS_Library:LED_D3.0mm; symbol GEMS_library:LED -> GEMS_Library:LED
- J1: footprint GEMS_library:USB-C_MOLEX-216990-0001 -> GEMS_Library:USB-C_MOLEX-216990-0001; symbol GEMS_library:USB_C_USB2.0 -> GEMS_Library:USB_C_USB2.0
- J2: footprint GEMS_library:18650_battery_holder -> GEMS_Library:18650_battery_holder; symbol GEMS_library:18650_battery_holder -> GEMS_Library:18650_battery_holder
- Q1: footprint GEMS_library:SOT-23 -> GEMS_Library:SOT-23; symbol GEMS_library:DMG2305UX-13 -> GEMS_Library:DMG2305UX-13
- Q2: footprint GEMS_library:SOIC-8 -> GEMS_Library:SOIC-8; symbol GEMS_library:DMP3036SSD-13 -> GEMS_Library:DMP3036SSD-13
- Q3, Q4: footprint GEMS_library:SOT-23 -> GEMS_Library:SOT-23; symbol GEMS_library:BC846 -> GEMS_Library:BC846
- Q5: footprint GEMS_library:SOT-23 -> GEMS_Library:SOT-23; symbol GEMS_library:DMN2310U -> GEMS_Library:DMN2310U
- R1, R10, R11, R12, R13, R14, R15, R16, R17, R18, R19, R2, R20, R21, R22, R23, R24, R25, R26, R27, R28, R29, R3, R30, R31, R4, R5, R6, R7, R8, R9: footprint GEMS_library:R_1206_(3216) -> GEMS_Library:R_1206_(3216); symbol GEMS_library:Resistor -> GEMS_Library:Resistor
- SW1, SW2, SW3: footprint GEMS_library:SW_PUSH_6mm_SMD -> GEMS_Library:SW_PUSH_6mm_SMD; symbol GEMS_library:SW_Push_NO -> GEMS_Library:SW_Push_NO
- SW4: footprint GEMS_library:SW_SPDT -> GEMS_Library:SW_SPDT; symbol GEMS_library:SW_SPDT -> GEMS_Library:SW_SPDT
- U1: footprint GEMS_library:SOT-89-5 -> GEMS_Library:SOT-89-5; symbol GEMS_library:R1170H331B -> GEMS_Library:R1170H331B
- U2: footprint GEMS_library:ESP32-C3-WROOM-02 -> GEMS_Library:ESP32-C3-WROOM-02; symbol GEMS_library:ESP32-C3 -> GEMS_Library:ESP32-C3
- U3: footprint GEMS_library:SOT-23-6 -> GEMS_Library:SOT-23-6; symbol GEMS_library:USBLC6-2SC6 -> GEMS_Library:USBLC6-2SC6
- U4: footprint GEMS_library:SOIC-8 -> GEMS_Library:SOIC-8; symbol GEMS_library:MCP6002 -> GEMS_Library:MCP6002
- U5: footprint GEMS_library:SOT-23-5 -> GEMS_Library:SOT-23-5; symbol GEMS_library:MCP73831T -> GEMS_Library:MCP73831T
- U6: footprint GEMS_library:SOIC-8 -> GEMS_Library:SOIC-8; symbol GEMS_library:TCAN332DR -> GEMS_Library:TCAN332DR
