File: GEMS_Ruby/GEMS_Ruby.kicad_pcb (KiCad board)
At the start: 2 copper layers, 90 x 40 mm, 70 parts, among them J1 USB_C_USB2.0, Q1 DMG2305UX-13, SW1 BTN, SW2 RST, U1 R1170H331B, U2 ESP32-C3, U3 USBLC6-2SC6, U4 MAX4468, U5 MAX4468, U6 RCWL-1601, U7 TCAN332DR

Commit message: updated Library
Parts:
- C1, C10, C11, C12, C13, C14, C15, C16, C17, C18, C19, C2, C20, C3, C4, C5, C6, C7, C8, C9: footprint GEMS_library:C_1206_(3216) -> GEMS_Library:C_1206_(3216)
- CAN1, CAN2: footprint GEMS_library:IDC8_Micro-MaTch -> GEMS_Library:IDC8_Micro-MaTch
- D1: footprint GEMS_library:DO-214_(SMA) -> GEMS_Library:DO-214_(SMA)
- D2, D3, D4, D5, D6, D7, D8: footprint GEMS_library:LED_D3.0mm -> GEMS_Library:LED_D3.0mm
- J1: footprint GEMS_library:USB-C_MOLEX-216990-0001 -> GEMS_Library:USB-C_MOLEX-216990-0001
- MIC1, MIC2: footprint GEMS_library:CMA-4544PF-W -> GEMS_Library:CMA-4544PF-W
- Q1: footprint GEMS_library:SOT-23 -> GEMS_Library:SOT-23
- R1, R10, R11, R12, R13, R14, R15, R16, R17, R18, R19, R2, R20, R21, R22, R23, R24, R25, R26, R3, R4, R5, R6, R7, R8, R9: footprint GEMS_library:R_1206_(3216) -> GEMS_Library:R_1206_(3216)
- SW1, SW2: footprint GEMS_library:SW_PUSH_6mm_SMD -> GEMS_Library:SW_PUSH_6mm_SMD
- U1: footprint GEMS_library:SOT-89-5 -> GEMS_Library:SOT-89-5
- U2: footprint GEMS_library:ESP32-C3-WROOM-02 -> GEMS_Library:ESP32-C3-WROOM-02
- U3: footprint GEMS_library:SOT-23-6 -> GEMS_Library:SOT-23-6
- U4, U5: footprint GEMS_library:SOT-23-8 -> GEMS_Library:SOT-23-8
- U6: footprint GEMS_library:RCWL-1601 -> GEMS_Library:RCWL-1601
- U7: footprint GEMS_library:SOIC-8 -> GEMS_Library:SOIC-8
