File: GEMS_Ruby/GEMS_Ruby.kicad_sch (KiCad schematic)
At the start: 69 parts, among them J1 USB_C_USB2.0, Q1 DMG2305UX-13, SW1 BTN, SW2 RST, U1 R1170H331B, U2 ESP32-C3, U3 USBLC6-2SC6, U4 MAX4468, U5 MAX4468, U6 RCWL-1601, U7 TCAN332DR

Commit message: updated Library
Parts:
- C1, C10, C11, C12, C13, C14, C15, C16, C17, C18, C19, C2, C20, C3, C4, C5, C6, C7, C8, C9: footprint GEMS_library:C_1206_(3216) -> GEMS_Library:C_1206_(3216); symbol GEMS_library:Capacitor -> GEMS_Library:Capacitor
- CAN1, CAN2: footprint GEMS_library:IDC8_Micro-MaTch -> GEMS_Library:IDC8_Micro-MaTch; symbol GEMS_library:CAN_connector -> GEMS_Library:CAN_connector
- D1: footprint GEMS_library:DO-214_(SMA) -> GEMS_Library:DO-214_(SMA); symbol GEMS_library:XBS306 -> GEMS_Library:XBS306
- D2, D3, D4, D5, D6, D7, D8: footprint GEMS_library:LED_D3.0mm -> GEMS_Library:LED_D3.0mm; symbol GEMS_library:LED -> GEMS_Library:LED
- J1: footprint GEMS_library:USB-C_MOLEX-216990-0001 -> GEMS_Library:USB-C_MOLEX-216990-0001; symbol GEMS_library:USB_C_USB2.0 -> GEMS_Library:USB_C_USB2.0
- MIC1, MIC2: footprint GEMS_library:CMA-4544PF-W -> GEMS_Library:CMA-4544PF-W; symbol GEMS_library:CMA-4544PF-W -> GEMS_Library:CMA-4544PF-W
- Q1: footprint GEMS_library:SOT-23 -> GEMS_Library:SOT-23; symbol GEMS_library:DMG2305UX-13 -> GEMS_Library:DMG2305UX-13
- R1, R10, R11, R12, R13, R14, R15, R16, R17, R18, R19, R2, R20, R21, R22, R23, R24, R25, R26, R3, R4, R5, R6, R7, R8, R9: footprint GEMS_library:R_1206_(3216) -> GEMS_Library:R_1206_(3216); symbol GEMS_library:Resistor -> GEMS_Library:Resistor
- SW1, SW2: footprint GEMS_library:SW_PUSH_6mm_SMD -> GEMS_Library:SW_PUSH_6mm_SMD; symbol GEMS_library:SW_Push_NO -> GEMS_Library:SW_Push_NO
- U1: footprint GEMS_library:SOT-89-5 -> GEMS_Library:SOT-89-5; symbol GEMS_library:R1170H331B -> GEMS_Library:R1170H331B
- U2: footprint GEMS_library:ESP32-C3-WROOM-02 -> GEMS_Library:ESP32-C3-WROOM-02; symbol GEMS_library:ESP32-C3 -> GEMS_Library:ESP32-C3
- U3: footprint GEMS_library:SOT-23-6 -> GEMS_Library:SOT-23-6; symbol GEMS_library:USBLC6-2SC6 -> GEMS_Library:USBLC6-2SC6
- U4, U5: footprint GEMS_library:SOT-23-8 -> GEMS_Library:SOT-23-8; symbol GEMS_library:MAX4468 -> GEMS_Library:MAX4468
- U6: footprint GEMS_library:RCWL-1601 -> GEMS_Library:RCWL-1601; symbol GEMS_library:RCWL-1601 -> GEMS_Library:RCWL-1601
- U7: footprint GEMS_library:SOIC-8 -> GEMS_Library:SOIC-8; symbol GEMS_library:TCAN332DR -> GEMS_Library:TCAN332DR
