File: GEMS_Sapphire/GEMS_Sapphire.kicad_sch (KiCad schematic)
At the start: 36 parts, among them J1 USB_C_USB2.0, J2 Conn_01x04, J3 I2C, Q1 DMG2305UX-13, SW1 BTN, SW2 RST, SW3 USR, U1 R1170H331B, U2 ESP32-S3-WROOM, U3 USBLC6-2SC6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

Commit message: updated Library
Parts:
- BZ1: footprint GEMS_library:CPT-1117-83-SMT -> GEMS_Library:CPT-1117-83-SMT; symbol GEMS_library:Buzzer -> GEMS_Library:Buzzer
- C1, C2, C3, C4, C5, C6, C7, C8, C9: footprint GEMS_library:C_1206_(3216) -> GEMS_Library:C_1206_(3216); symbol GEMS_library:Capacitor -> GEMS_Library:Capacitor
- CAN1, CAN2: footprint GEMS_library:IDC8_Micro-MaTch -> GEMS_Library:IDC8_Micro-MaTch; symbol GEMS_library:CAN_connector -> GEMS_Library:CAN_connector
- D1: footprint GEMS_library:DO-214_(SMA) -> GEMS_Library:DO-214_(SMA); symbol GEMS_library:XBS306 -> GEMS_Library:XBS306
- D2: footprint GEMS_library:LED_D3.0mm -> GEMS_Library:LED_D3.0mm; symbol GEMS_library:LED -> GEMS_Library:LED
- Displ1: footprint GEMS_library:MDOB128032GV-WI -> GEMS_Library:MDOB128032GV-WI; symbol GEMS_library:OLED_Display_I2C -> GEMS_Library:OLED_Display_I2C
- J1: footprint GEMS_library:USB-C_MOLEX-216990-0001 -> GEMS_Library:USB-C_MOLEX-216990-0001; symbol GEMS_library:USB_C_USB2.0 -> GEMS_Library:USB_C_USB2.0
- J2, J3: footprint GEMS_library:PinHeader_1x04_P2.54mm_Vertical -> GEMS_Library:PinHeader_1x04_P2.54mm_Vertical; symbol GEMS_library:Conn_01x04 -> GEMS_Library:Conn_01x04
- Q1: footprint GEMS_library:SOT-23 -> GEMS_Library:SOT-23; symbol GEMS_library:DMG2305UX-13 -> GEMS_Library:DMG2305UX-13
- R1, R10, R2, R3, R4, R5, R6, R7, R8, R9: footprint GEMS_library:R_1206_(3216) -> GEMS_Library:R_1206_(3216); symbol GEMS_library:Resistor -> GEMS_Library:Resistor
- SW1, SW2, SW3: footprint GEMS_library:SW_PUSH_6mm_SMD -> GEMS_Library:SW_PUSH_6mm_SMD; symbol GEMS_library:SW_Push_NO -> GEMS_Library:SW_Push_NO
- U1: footprint GEMS_library:SOT-89-5 -> GEMS_Library:SOT-89-5; symbol GEMS_library:R1170H331B -> GEMS_Library:R1170H331B
- U2: footprint GEMS_library:ESP32-S3-WROOM -> GEMS_Library:ESP32-S3-WROOM; symbol GEMS_library:ESP32-S3-WROOM -> GEMS_Library:ESP32-S3-WROOM
- U3: footprint GEMS_library:SOT-23-6 -> GEMS_Library:SOT-23-6; symbol GEMS_library:USBLC6-2SC6 -> GEMS_Library:USBLC6-2SC6
- U4: footprint GEMS_library:SOIC-8 -> GEMS_Library:SOIC-8; symbol GEMS_library:TCAN332DR -> GEMS_Library:TCAN332DR
